Commit message: working commit of heron in vrx

File: heron_description/urdf/base.xacro (robot description, xacro)
@@ -10,4 +10,5 @@
   <xacro:property name="rho" value="1028"/>
   <!-- Loading vehicle's specific macros -->
+  <!-- TODO -->
   <xacro:include filename="$(find heron_description)/urdf/snippets.xacro"/>
   <material name="gray"><color rgba="0.7 0.7 0.7 1.0"/></material>
@@ -95,4 +96,76 @@
       <origin xyz="-0.53 0.377654 -0.16" rpy="0 0 0" />
     </xacro:thruster_macro>s
+    <!-- TODO -->
+    <gazebo>
+      <!-- USV Gazebo Thrust plugin -->
+        <plugin name="$(arg namespace)_thruster_model" filename="libusv_gazebo_thrust_plugin.so">
+        <!-- General plugin parameters -->
+        <robotNamespace>$(arg namespace)"</robotNamespace>
+        <cmdTimeout>1.0</cmdTimeout>
+        <publisherRate>100.0></publisherRate>
+        <!-- Two thrusters -->
+        <thruster>
+          <linkName>$(arg suffix_ns)thruster_0</linkName>
+          <!-- TODO -->
+          <!-- propJointName dummy/empty since heron uses jets -->
+          <propJointName>$(arg suffix_ns)thruster_0_joint</propJointName>
+          <!-- engineJointName dummy/empty since heron uses jets -->
+          <engineJointName>$(arg suffix_ns)thruster_0_joint</engineJointName>
+          <cmdTopic>"$(arg suffix_ns)/thruster_0/input"</cmdTopic>
+          <!-- angleTopic empty since heron uses jets -->
+          <angleTopic></angleTopic>
+          <!-- enableAngle false since heron uses jets -->
+          <enableAngle>false</enableAngle>
+          <mappingType>1</mappingType>
+          <maxCmd>100</maxCmd>
+          <maxForceFwd>35</maxForceFwd>
+          <maxForceRev>-35</maxForceRev>
+          <!-- maxAngle of 0 since heron uses jets -->
+          <maxAngle>0</maxAngle>
+        </thruster>
+        <thruster>
+          <linkName>$(arg suffix_ns)thruster_1</linkName>
+          <!-- TODO -->
+          <!-- propJointName dummy/empty since heron uses jets -->
+          <propJointName>$(arg suffix_ns)thruster_1_joint</propJointName>
+          <!-- engineJointName dummy/empty since heron uses jets -->
+          <engineJointName>$(arg suffix_ns)thruster_1_joint</engineJointName>
+          <cmdTopic>"$(arg suffix_ns)/thruster_1/input"</cmdTopic>
+          <!-- angleTopic empty since heron uses jets -->
+          <angleTopic></angleTopic>
+          <!-- enableAngle false since heron uses jets -->
+          <enableAngle>false</enableAngle>
+          <mappingType>1</mappingType>
+          <maxCmd>100</maxCmd>
+          <maxForceFwd>35</maxForceFwd>
+          <maxForceRev>-35</maxForceRev>
+          <!-- maxAngle of 0 since heron uses jets -->
+          <maxAngle>0</maxAngle>
+        </thruster>
+        <!-- Name of the joint between thruster and vehicle base link -->
+        <!--jointName>${suffix_ns}thruster_${thruster_id}_joint</jointName-->
+        <!-- FIXME: skip for now -->
+        <!-- Minimum allowed value for the input signal for thruster unit -->
+        <clampMin>-100</clampMin>
+        <!-- FIXME: skip for now -->
+        <!-- 2) First order model -->
+        <dynamics>
+          <type>FirstOrder</type>
+          <timeConstant>0.05</timeConstant>
+        </dynamics>
+        <!-- FIXME: skip for now -->
+        <!-- 3) Linear interpolation
+        If you have access to the thruster's data sheet, for example,
+        you can enter samples of the curve's input and output values
+        and the thruster output will be found through linear interpolation
+        of the given samples.
+        -->
+        <conversion>
+          <type>LinearInterp</type>
+          <inputValues>-1.0 -0.8 -0.6 -0.4 -0.2 0 0.2 0.4 0.6 0.8 1.0</inputValues>
+          <outputValues>-19.88 -16.52 -12.6 -5.6 -1.4 0.0 2.24 9.52 21.28 28.0 33.6</outputValues>
+        </conversion>
+      </plugin>
+    </gazebo>
     <!-- Include the sensor modules -->
     <xacro:include filename="$(find heron_description)/urdf/sensors.xacro"/>

File: heron_description/urdf/gazebo.xacro (robot description, xacro)
@@ -1,62 +1,39 @@
 <?xml version="1.0"?>
 <robot xmlns:xacro="http://www.ros.org/wiki/xacro">
-    <!-- Center of buoyancy -->
-    <xacro:property name="heron_cob" value="0 0 0"/>
-    <!-- Vehicle's actual volume (Gazebo cannot compute the volume out of the mesh) -->
-    <xacro:property name="heron_volume" value="0.13"/>
-    <!-- Describing the dimensions of the vehicle's bounding box -->
-    <xacro:property name="heron_length" value="1.35"/>
-    <xacro:property name="heron_width"  value="1.0"/>
-    <xacro:property name="heron_height" value="0.32"/>
     <xacro:macro name="heron_hydro_model" params="namespace">
-      <!-- List of hydrodynamic models this robot's links -->
-      <link name="${namespace}base_link">
-              <volume>${heron_volume}</volume>
-              <box>
-                  <width>${heron_width}</width>
-                  <length>${heron_length}</length>
-                  <height>${heron_height}</height>
-              </box>
-              <center_of_buoyancy>${heron_cob}</center_of_buoyancy>
-              <!-- The buoyancy plugin in the UUV Simulator can then be adapted
-                   to receive the additional parameters used to describe the
-                   buoyancy force computation for the surface vessel.
-              -->
-              <metacentric_width>0.1</metacentric_width>
-              <metacentric_length>0.1</metacentric_length>
-              <submerged_height>0.02</submerged_height>
-              <hydrodynamic_model>
-                  <type>fossen</type>
-                  <added_mass>
-                     0   0   0   0   0   0
-                     0   0   0   0   0   0
-                     0   0   0   0   0   0
-                     0   0   0   0   0   0
-                     0   0   0   0   0   0
-                     0   0   0   0   0   0
-                </added_mass>
-                <offset_added_mass>0</offset_added_mass>
-                  <linear_damping>
-                      -16.44998712 -15.79776044 -100 -13 -13 -6
-                  </linear_damping>
-                  <quadratic_damping>
-                    -2.942 -2.7617212 -10 -5 -5 -5
-                  </quadratic_damping>
-                  <!-- Sanity check -->
-                  <linear_damping_forward_speed>
-                    0 0 0 0 0 0
-                  </linear_damping_forward_speed>
-                  <offset_linear_damping>
-                    0
-                  </offset_linear_damping>
-                  <offset_lin_forward_speed_damping>
-                    0
-                  </offset_lin_forward_speed_damping>
-                  <offset_nonlin_damping>
-                    0
-                  </offset_nonlin_damping>
-                  <scaling_damping>1.0</scaling_damping>
-              </hydrodynamic_model>
-          </link>
+      <bodyName>${namespace}base_link</bodyName>
+      <!-- Must be same as the ocean model!-->
+      <waterLevel>0</waterLevel>
+      <waterDensity>997.8</waterDensity>
+      <!-- Added mass -->
+      <xDotU>0</xDotU>
+      <yDotV>0</yDotV>
+      <zDotW>0</zDotW>
+      <kDotP>0</kDotP>
+      <kDotP>0</kDotP>
+      <mDotQ>0</mDotQ>
+      <nDotR>0</nDotR>
+      <!-- Linear and quadratic drag -->
+      <xU>16.44998712</xU>
+      <xUU>2.942</xUU>
+      <yV>15.79776044</yV>
+      <yVV>2.7617212</yVV>
+      <zW>100</zW>
+      <zWW>10</zWW>
+      <kP>13</kP>
+      <kPP>5</kPP>
+      <mQ>13</mQ>
+      <mQQ>5</mQQ>
+      <nR>6</nR>
+      <nRR>5</nRR>
+      <!-- General dimensions -->
+      <!-- TODO: hullRadius is an estimation -->
+      <hullRadius>0.15</hullRadius>
+      <boatWidth>1.0</boatWidth>
+      <boatLength>1.35</boatLength>
+      <!-- Length discretization, AKA, "N" -->
+      <length_n>2</length_n>
+      <!-- Wave model -->
+      <wave_model>ocean_waves</wave_model>
     </xacro:macro>
 </robot>

File: heron_description/urdf/heron.urdf.xacro (robot description, xacro)
@@ -26,5 +26,4 @@
 -->
 <robot name="heron" xmlns:xacro="http://www.ros.org/wiki/xacro" >
-  <xacro:arg name="debug" default="0"/>
   <xacro:arg name="namespace" default=""/>
   <xacro:arg name="suffix_ns" default="$(arg namespace)"/>
@@ -34,29 +33,10 @@
   <!-- Create the heron -->
   <xacro:heron_base namespace="$(arg suffix_ns)">
-    <!-- The underwater object plugin is given as an input block parameter to
-     allow the addition of external models of manipulator units -->
     <gazebo>
-      <plugin name="uuv_plugin" filename="libuuv_underwater_object_ros_plugin.so">
-        <fluid_density>1028.0</fluid_density>
-        <flow_velocity_topic>hydrodynamics/current_velocity</flow_velocity_topic>
-        <debug>$(arg debug)</debug>
-        <!-- Adding the hydrodynamic and hydrostatic parameters for the vehicle-->
+      <plugin name="usv_dynamics_heron" filename="libusv_gazebo_dynamics_plugin.so">
         <xacro:heron_hydro_model namespace="$(arg suffix_ns)" />
-        <!--
-          In case other modules are added to the vehicle (such as a manipulator)
-          that also have link running with the underwater object plugin, they
-          should also be added in this block. For this, this new module should
-          have a file similar to gazebo.xacro above with the description of the
-          parameter necessary for the underwater object plugin to be initialized.
-        -->
       </plugin>
     </gazebo>
   </xacro:heron_base>
-  <!-- Joint state publisher plugin -->
-  <gazebo>
-    <plugin name="joint_state_publisher" filename="libuuv_joint_state_publisher.so">
-      <robotNamespace>/$(arg namespace)</robotNamespace>
-      <updateRate>10</updateRate>
-    </plugin>
-  </gazebo>
+  <!-- TODO do we need a joint state publisher?-->
 </robot>

File: heron_description/urdf/snippets.xacro (robot description, xacro)
@@ -34,52 +34,4 @@
         <child link="${suffix_ns}thruster_${thruster_id}" />
       </joint>
-      <gazebo>
-        <!-- Thruster ROS plugin -->
-        <plugin name="${robot_namespace}thruster_${thruster_id}_thruster_model" filename="libuuv_thruster_ros_plugin.so">
-          <!-- Name of the thruster link -->
-          <linkName>${suffix_ns}thruster_${thruster_id}</linkName>
-          <!-- Name of the joint between thruster and vehicle base link -->
-          <jointName>${suffix_ns}thruster_${thruster_id}_joint</jointName>
-          <!-- Make the thruster aware of its id -->
-          <thrusterID>${thruster_id}</thrusterID>
-          <!-- Gain of the input command signal -->
-          <gain>1</gain>
-          <!-- Maximum allowed input value for the input signal for thruster unit -->
-          <clampMax>100</clampMax>
-          <!-- Minimum allowed value for the input signal for thruster unit -->
-          <clampMin>-100</clampMin>
-          <!-- Minimum and maximum thrust force output allowed -->
-          <thrustMin>-35</thrustMin>
-          <thrustMax>35</thrustMax>
-          <!--
-          Value from 0 to 1 to set the efficiency of the output thrust force
-          Default value is 1.0
-          -->
-          <thrust_efficiency>1</thrust_efficiency>
-          <!--
-          Value from 0 to 1 to set the efficiency of the propeller as a factor
-          to be multiplied to the current value of the state variable at each
-          iteration.
-          Default value is 1.0
-          -->
-          <propeller_efficiency>1</propeller_efficiency>
-          <!-- 2) First order model -->
-          <dynamics>
-            <type>FirstOrder</type>
-            <timeConstant>0.05</timeConstant>
-          </dynamics>
-          <!-- 3) Linear interpolation
-          If you have access to the thruster's data sheet, for example,
-          you can enter samples of the curve's input and output values
-          and the thruster output will be found through linear interpolation
-          of the given samples.
-          -->
-          <conversion>
-            <type>LinearInterp</type>
-            <inputValues>-1.0 -0.8 -0.6 -0.4 -0.2 0 0.2 0.4 0.6 0.8 1.0</inputValues>
-            <outputValues>-19.88 -16.52 -12.6 -5.6 -1.4 0.0 2.24 9.52 21.28 28.0 33.6</outputValues>
-          </conversion>
-        </plugin>
-      </gazebo>
       <gazebo reference="${suffix_ns}thruster_${thruster_id}">
         <selfCollide>false</selfCollide>

Commit message: fix usage of usv thruster plugin

File: heron_description/urdf/base.xacro (robot description, xacro)
@@ -10,5 +10,4 @@
   <xacro:property name="rho" value="1028"/>
   <!-- Loading vehicle's specific macros -->
-  <!-- TODO -->
   <xacro:include filename="$(find heron_description)/urdf/snippets.xacro"/>
   <material name="gray"><color rgba="0.7 0.7 0.7 1.0"/></material>
@@ -86,4 +85,5 @@
     <xacro:insert_block name="gazebo"/>
     <!-- Include the thruster modules -->
+    <!-- See: osrf/vrx/wamv_gazebo/urdf/thruster_layouts/wamv_aft_thrusters.xacro -->
     <xacro:thruster_macro robot_namespace="$(arg namespace)" suffix_ns="$(arg suffix_ns)" thruster_id="0"
       simulation="$(arg simulation)">
@@ -96,10 +96,9 @@
       <origin xyz="-0.53 0.377654 -0.16" rpy="0 0 0" />
     </xacro:thruster_macro>s
-    <!-- TODO -->
     <gazebo>
       <!-- USV Gazebo Thrust plugin -->
-        <plugin name="$(arg namespace)_thruster_model" filename="libusv_gazebo_thrust_plugin.so">
+      <plugin name="heron_thruster_model" filename="libusv_gazebo_thrust_plugin.so">
         <!-- General plugin parameters -->
-        <robotNamespace>$(arg namespace)"</robotNamespace>
+        <robotNamespace>$(arg namespace)</robotNamespace>
         <cmdTimeout>1.0</cmdTimeout>
         <publisherRate>100.0></publisherRate>
@@ -107,63 +106,36 @@
         <thruster>
           <linkName>$(arg suffix_ns)thruster_0</linkName>
-          <!-- TODO -->
-          <!-- propJointName dummy/empty since heron uses jets -->
-          <propJointName>$(arg suffix_ns)thruster_0_joint</propJointName>
-          <!-- engineJointName dummy/empty since heron uses jets -->
-          <engineJointName>$(arg suffix_ns)thruster_0_joint</engineJointName>
-          <cmdTopic>"$(arg suffix_ns)/thruster_0/input"</cmdTopic>
-          <!-- angleTopic empty since heron uses jets -->
+          <propJointName>$(arg suffix_ns)thruster_0_engine_propeller_joint</propJointName>
+          <engineJointName>$(arg suffix_ns)thruster_0_chassis_engine_joint</engineJointName>
+          <cmdTopic>$(arg suffix_ns)thrusters/0/input</cmdTopic>
+          <!-- angleTopic empty since heron cannot rotate it's engine -->
           <angleTopic></angleTopic>
-          <!-- enableAngle false since heron uses jets -->
+          <!-- enableAngle false since heron cannot rotate it's engine -->
           <enableAngle>false</enableAngle>
-          <mappingType>1</mappingType>
-          <maxCmd>100</maxCmd>
-          <maxForceFwd>35</maxForceFwd>
-          <maxForceRev>-35</maxForceRev>
-          <!-- maxAngle of 0 since heron uses jets -->
+          <mappingType>0</mappingType>
+          <maxCmd>1</maxCmd>
+          <minCmd>-1</minCmd>
+          <maxForceFwd>45</maxForceFwd>
+          <maxForceRev>-25</maxForceRev>
+          <!-- maxAngle of 0 since heron cannot rotate it's engine -->
           <maxAngle>0</maxAngle>
         </thruster>
         <thruster>
           <linkName>$(arg suffix_ns)thruster_1</linkName>
-          <!-- TODO -->
-          <!-- propJointName dummy/empty since heron uses jets -->
-          <propJointName>$(arg suffix_ns)thruster_1_joint</propJointName>
-          <!-- engineJointName dummy/empty since heron uses jets -->
-          <engineJointName>$(arg suffix_ns)thruster_1_joint</engineJointName>
-          <cmdTopic>"$(arg suffix_ns)/thruster_1/input"</cmdTopic>
-          <!-- angleTopic empty since heron uses jets -->
+          <propJointName>$(arg suffix_ns)thruster_1_engine_propeller_joint</propJointName>
+          <engineJointName>$(arg suffix_ns)thruster_1_chassis_engine_joint</engineJointName>
+          <cmdTopic>$(arg suffix_ns)thrusters/1/input</cmdTopic>
+          <!-- angleTopic empty since heron cannot rotate it's engine -->
           <angleTopic></angleTopic>
-          <!-- enableAngle false since heron uses jets -->
+          <!-- enableAngle false since heron cannot rotate it's engine -->
           <enableAngle>false</enableAngle>
-          <mappingType>1</mappingType>
-          <maxCmd>100</maxCmd>
-          <maxForceFwd>35</maxForceFwd>
-          <maxForceRev>-35</maxForceRev>
-          <!-- maxAngle of 0 since heron uses jets -->
+          <mappingType>0</mappingType>
+          <maxCmd>1</maxCmd>
+          <minCmd>-1</minCmd>
+          <maxForceFwd>45</maxForceFwd>
+          <maxForceRev>-25</maxForceRev>
+          <!-- maxAngle of 0 since heron cannot rotate it's engine -->
           <maxAngle>0</maxAngle>
         </thruster>
-        <!-- Name of the joint between thruster and vehicle base link -->
-        <!--jointName>${suffix_ns}thruster_${thruster_id}_joint</jointName-->
-        <!-- FIXME: skip for now -->
-        <!-- Minimum allowed value for the input signal for thruster unit -->
-        <clampMin>-100</clampMin>
-        <!-- FIXME: skip for now -->
-        <!-- 2) First order model -->
-        <dynamics>
-          <type>FirstOrder</type>
-          <timeConstant>0.05</timeConstant>
-        </dynamics>
-        <!-- FIXME: skip for now -->
-        <!-- 3) Linear interpolation
-        If you have access to the thruster's data sheet, for example,
-        you can enter samples of the curve's input and output values
-        and the thruster output will be found through linear interpolation
-        of the given samples.
-        -->
-        <conversion>
-          <type>LinearInterp</type>
-          <inputValues>-1.0 -0.8 -0.6 -0.4 -0.2 0 0.2 0.4 0.6 0.8 1.0</inputValues>
-          <outputValues>-19.88 -16.52 -12.6 -5.6 -1.4 0.0 2.24 9.52 21.28 28.0 33.6</outputValues>
-        </conversion>
       </plugin>
     </gazebo>

File: heron_description/urdf/gazebo.xacro (robot description, xacro)
@@ -38,5 +38,5 @@
         <link_name>${namespace}/base_link</link_name>
         <geometry>
-          <mesh filename="package://heron_description/meshes/only_hull.stl"/>
+          <mesh filename="package://heron_description/meshes/heron_collision.stl"/>
         </geometry>
       </buoyancy>

File: heron_description/urdf/snippets.xacro (robot description, xacro)
@@ -7,4 +7,18 @@
   -->
   <xacro:macro name="thruster_macro" params="robot_namespace suffix_ns thruster_id *origin simulation:=false">
+    <!--
+    Dummy link as place holder for the engine frame,
+    since vrx usv_thrust_plugin requires an engine link that can orient the
+    propeller/thruster
+    -->
+    <link name="${suffix_ns}thruster_${thruster_id}_engine_link">
+      <inertial>
+        <mass value="0.001" />
+        <origin xyz="0 0 0" rpy="0 0 0"/>
+        <inertia ixx="0.000000017" ixy="0.0" ixz="0.0"
+               iyy="0.000000017" iyz="0.0"
+               izz="0.000000017" />
+      </inertial>
+    </link>
     <!--
     Dummy link as place holder for the thruster frame,
@@ -27,6 +41,13 @@
     </link>
     <xacro:if value="${simulation}">
-      <!-- Joint between thruster link and vehicle base link -->
-      <joint name="${suffix_ns}thruster_${thruster_id}_joint" type="continuous">
+      <!-- Dummy engine joint for angle command between thruster link and vehicle base link -->
+      <joint name="${suffix_ns}thruster_${thruster_id}_chassis_engine_joint" type="revolute">
+        <!--xacro:insert_block name="origin" /-->
+        <limit lower="0" upper="0" effort="0" velocity="0"/>
+        <parent link="${suffix_ns}base_link" />
+        <child link="${suffix_ns}thruster_${thruster_id}_engine_link" />
+      </joint>
+      <!-- Propeller joint for force command between thruster link and vehicle base link -->
+      <joint name="${suffix_ns}thruster_${thruster_id}_engine_propeller_joint" type="continuous">
         <xacro:insert_block name="origin" />
         <axis xyz="1 0 0" />
@@ -34,4 +55,7 @@
         <child link="${suffix_ns}thruster_${thruster_id}" />
       </joint>
+      <gazebo reference="${suffix_ns}thruster_${thruster_id}_engine_link">
+        <selfCollide>false</selfCollide>
+      </gazebo>
       <gazebo reference="${suffix_ns}thruster_${thruster_id}">
         <selfCollide>false</selfCollide>
@@ -39,8 +63,14 @@
     </xacro:if>
     <xacro:unless value="${simulation}">
-      <!-- On the real robot this joint is purely decorative; it's only used to produce thrust in gazebo -->
-      <joint name="${suffix_ns}thruster_${thruster_id}_joint" type="fixed">
+      <!-- Dummy engine joint for angle command between thruster link and vehicle base link -->
+      <joint name="${suffix_ns}thruster_${thruster_id}_chassis_engine_joint" type="fixed">
         <xacro:insert_block name="origin" />
         <parent link="${suffix_ns}base_link" />
+        <child link="${suffix_ns}thruster_${thruster_id}_engine_link" />
+      </joint>
+      <!-- On the real robot this joint is purely decorative; it's only used to produce thrust in gazebo -->
+      <joint name="${suffix_ns}thruster_${thruster_id}_engine_propeller_joint" type="fixed">
+        <xacro:insert_block name="origin" />
+        <parent link="${suffix_ns}thruster_${thruster_id}_engine_link" />
         <child link="${suffix_ns}thruster_${thruster_id}" />
       </joint>
