Commit message: use mesh buoyancy with vrx surface geom branch

File: heron_description/urdf/gazebo.xacro (robot description, xacro)
@@ -2,5 +2,5 @@
 <robot xmlns:xacro="http://www.ros.org/wiki/xacro">
     <xacro:macro name="heron_hydro_model" params="namespace">
-      <bodyName>${namespace}base_link</bodyName>
+      <bodyName>${namespace}/base_link</bodyName>
       <!-- Must be same as the ocean model!-->
       <waterLevel>0</waterLevel>
@@ -27,13 +27,18 @@
       <nR>6</nR>
       <nRR>5</nRR>
-      <!-- General dimensions -->
-      <!-- TODO: hullRadius is an estimation -->
-      <hullRadius>0.15</hullRadius>
-      <boatWidth>1.0</boatWidth>
-      <boatLength>1.35</boatLength>
-      <!-- Length discretization, AKA, "N" -->
-      <length_n>2</length_n>
+    </xacro:macro>
+    <xacro:macro name="heron_buoyancy_model" params="namespace">
       <!-- Wave model -->
       <wave_model>ocean_waves</wave_model>
+      <fluid_density>997.8</fluid_density>
+      <fluid_level>0</fluid_level>
+      <linear_drag>0</linear_drag>
+      <angular_drag>0</angular_drag>
+      <buoyancy>
+        <link_name>${namespace}/base_link</link_name>
+        <geometry>
+          <mesh filename="package://heron_description/meshes/only_hull.stl"/>
+        </geometry>
+      </buoyancy>
     </xacro:macro>
 </robot>

File: heron_description/urdf/heron.urdf.xacro (robot description, xacro)
@@ -34,6 +34,11 @@
   <xacro:heron_base namespace="$(arg suffix_ns)">
     <gazebo>
+      <!--TODO(acxz): hardcoded namespace param to heron instead of $(arg suffix_ns)-->
       <plugin name="usv_dynamics_heron" filename="libusv_gazebo_dynamics_plugin.so">
-        <xacro:heron_hydro_model namespace="$(arg suffix_ns)" />
+        <xacro:heron_hydro_model namespace="heron" />
+      </plugin>
+      <!--TODO(acxz): hardcoded namespace param to heron instead of $(arg suffix_ns)-->
+      <plugin name="usv_buoyancy_heron" filename="libbuoyancy_gazebo_plugin.so">
+        <xacro:heron_buoyancy_model namespace="heron" />
       </plugin>
     </gazebo>

Commit message: use cylinder mesh for better sim and speed

File: heron_description/urdf/gazebo.xacro (robot description, xacro)
@@ -37,6 +37,20 @@
       <buoyancy>
         <link_name>${namespace}/base_link</link_name>
+        <pose>0 -0.5 -0.05 0 1.57 0</pose>
         <geometry>
-          <mesh filename="package://heron_description/meshes/heron_collision.stl"/>
+            <cylinder>
+                <radius>0.15</radius>
+                <length>1.35</length>
+            </cylinder>
+        </geometry>
+      </buoyancy>
+      <buoyancy>
+        <link_name>${namespace}/base_link</link_name>
+        <pose>0 0.5 -0.05 0 1.57 0</pose>
+        <geometry>
+            <cylinder>
+                <radius>0.15</radius>
+                <length>1.35</length>
+            </cylinder>
         </geometry>
       </buoyancy>
